File: pcb/func_amp.kicad_sch (KiCad schematic)
At the start: 44 parts, among them J1 L, J10 GNDS, J11 GND, J12 GNDPWR, J13 GNDPWR, J2 N, J3 G, J4 IN, J5 GNDS, J6 OUT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

Commit message: cleanup schematic
Other:
- note added: "size discharge resistors so no load votlage does not exceeded TDA2030 Vmax"
- note removed: "size discharge resistors so no load votlage does not exceeded tda2030 Vmax"
